File: PCB/TS06-FASCIA/TS06-FASCIA.kicad_sch (KiCad schematic)
At the start: 14 parts, among them J1 PH 6 SMT, SW1 SR25 6-pos, SW2 LEVER A, SW3 LEVER B, SW4 MINUS, SW5 PLUS

Commit message: sch: the panel connector symbol is JST-PH, not XH
The footprint, the buy list and the physical part have been PH 2.0 mm since the
connector was chosen. Only the symbol name still said XH, which is exactly the
kind of stale label that gets ordered against.

Co-Authored-By: Claude Opus 5 <noreply@anthropic.com>
Claude-Session: https://claude.ai/code/session_01Wbajb7CU1SV8ZUPn3KkB8i
Parts:
- removed J1: PH 6 SMT, TS06:TS06_JST_PH_S6B-PH-SM4-TB_Back, symbol TS06:Conn_JST_XH_6
- added J1: PH 6 SMT, TS06:TS06_JST_PH_S6B-PH-SM4-TB_Back, symbol TS06:Conn_JST_PH_6
Connections:
- net +5V: now also J1.1 (+5V)
- net A6: now also J1.3 (A6)
- net A7: now also J1.4 (A7)
- net D7: now also J1.5 (D7)
- net D8: now also J1.6 (D8)
- net GND: now also J1.2 (GND)
Changed lines of the file:
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@@
 )
 (symbol
-(lib_id "TS06:Conn_JST_XH_6")
+(lib_id "TS06:Conn_JST_PH_6")
 (at 238.76 80.01 0)
 (unit 1)
