File: PCB/TS06-MAIN-THT/TS06-MAIN-THT.kicad_sch (KiCad schematic)
At the start: 146 parts, among them J1 PH 6, U1 Arduino Nano, U10 TLP627, U11 TC4420, U12 LM393, U13 DS3231 mini, U14 R-78E5.0-1.0, U2 K155ID1, U3 MCP23017, U4 MCP23017, U5 TLP627, U6 TLP627, U7 TLP627, U8 TLP627, U9 TLP627

Commit message: sch: symbol libraries claim the library format version KiCad 10 writes
Both generators stamped the .kicad_sym files with the schematic format version
(20260306); KiCad 10.0.5 writes its own libraries as 20251024 and refuses to load a
library claiming a newer one, so the TS06 and TS06M libraries could not be opened in
the symbol editor and every schematic symbol raised a library warning in ERC. Fixed in
tools/mksch.py and tools/mksch_main.py, libraries and schematics regenerated; the two
main boards also get a KiCad project file so the library tables resolve.

Co-Authored-By: Claude Fable 5.1 <noreply@anthropic.com>
Parts:
- R1, R10, R11, R12, R13, R14, R15, R16, R17, R18, R19, R2, R20, R21, R22, R23, R24, R25, R26, R3, R33, R34, R35, R36, R37, R38, R39, R4, R40, R41, R42, R43, R44, R45, R46, R47, R48, R49, R5, R50, R51, R52, R53, R54, R55, R6, R60, R61, R62, R63, R64, R65, R66, R67, R68, R69, R7, R70, R71, R8, R9: footprint TS06:TS06_R_Axial_L6.3mm_P10.16mm_Back -> TS06:TS06_R_Axial_L6.3mm_P2.54mm_Vertical_Back
- R27, R28, R29, R30, R31, R32, R56, R57, R58, R59: footprint TS06:TS06_R_Axial_P12.7mm_Back -> TS06:TS06_R_Axial_L9.9mm_P5.08mm_Vertical_Back
