File: PCB/TS06-DRV-swap/TS06-DRV-swap.kicad_pcb (KiCad board)
At the start: 2 copper layers, 176 x 100 mm, 103 parts, among them J1 PH 6 vertical, U1 Arduino Nano, U10 TLP627, U11 TC4420, U12 LM393, U13 DS3231 mini, U14 R-78E5.0-1.0, U15 K155ID1, U16 K155ID1, U17 K155ID1, U2 K155ID1, U3 MCP23017-E/SP, U5 TLP627, U6 TLP627, U7 TLP627, U8 TLP627, U9 TLP627

Commit message: TS06-DRV swap: keep 185 V out of the logic strip (re-routed, converged, shorter); report updated
Co-Authored-By: Claude Opus 5.5 <noreply@anthropic.com>
Claude-Session: https://claude.ai/code/session_016UT9naQSnwzyf7HkDm2evf
Routing:
- net HV185: track 253.2 -> 227.3 mm
- net GND: track 615.5 -> 616.4 mm
Changed lines of the file:
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@@
 	(segment
 		(start 5.7 84)
-		(end 9.9 88.2)
+		(end 10 88.3)
 		(width 0.25)
 		(layer "B.Cu")
@@
 	)
 	(segment
-		(start 9.9 88.2)
-		(end 21.4 88.2)
+		(start 10 88.3)
+		(end 21.3 88.3)
 		(width 0.25)
 		(layer "B.Cu")
@@
 	)
 	(segment
-		(start 21.4 88.2)
+		(start 21.3 88.3)
 		(end 22 87.6)
 		(width 0.25)
@@
 	(segment
 		(start 79.5 48)
-		(end 80.1 47.4)
+		(end 80.2 47.3)
 		(width 0.25)
 		(layer "F.Cu")
@@
 	)
 	(segment
-		(start 80.1 47.4)
-		(end 90.7 47.4)
+		(start 80.2 47.3)
+		(end 90.8 47.3)
 		(width 0.25)
 		(layer "F.Cu")
@@
 	)
 	(segment
-		(start 90.7 47.4)
-		(end 97.2 53.9)
+		(start 90.8 47.3)
+		(end 97.3 53.8)
 		(width 0.25)
 		(layer "F.Cu")
@@
 	)
 	(segment
-		(start 97.2 53.9)
+		(start 97.3 53.8)
 		(end 97.4 54.54)
 		(width 0.25)
@@
 	)
 	(segment
-		(start 78.83 56.3)
-		(end 78.2 55.9)
-		(width 0.4)
-		(layer "F.Cu")
-		(net 80)
-	)
-	(segment
-		(start 78.2 55.9)
-		(end 78.2 53.1)
+		(start 84.63 56.3)
+		(end 85 56.9)
 		(width 0.4)
 		(layer "F.Cu")
@@
 	)
 	(segment
-		(start 78.2 53.1)
-		(end 74.5 49.4)
+		(start 85 56.9)
+		(end 112.1 56.9)
 		(width 0.4)
 		(layer "F.Cu")
@@
 	)
 	(segment
-		(start 74.5 49.4)
-		(end 74.5 46.1)
+		(start 112.1 56.9)
+		(end 113.2 58)
 		(width 0.4)
 		(layer "F.Cu")
@@
 	)
 	(segment
-		(start 74.5 46.1)
-		(end 91.4 46.1)
+		(start 113.2 58)
+		(end 115.4 58)
 		(width 0.4)
 		(layer "F.Cu")
@@
 	)
 	(segment
-		(start 91.4 46.1)
-		(end 95.3 50)
+		(start 115.4 58)
+		(end 116.5 56.9)
 		(width 0.4)
 		(layer "F.Cu")
@@
 	)
 	(segment
-		(start 95.3 50)
-		(end 110.8 50)
+		(start 116.5 56.9)
+		(end 116.88 56.3)
 		(width 0.4)
 		(layer "F.Cu")
@@
 	)
 	(segment
-		(start 110.8 50)
-		(end 116.5 55.7)
+		(start 116.88 56.3)
+		(end 117.3 55.7)
 		(width 0.4)
 		(layer "F.Cu")
@@
 	)
 	(segment
-		(start 116.5 55.7)
-		(end 116.88 56.3)
+		(start 117.3 55.7)
+		(end 118.5 54.5)
 		(width 0.4)
 		(layer "F.Cu")
@@
 	)
 	(segment
-		(start 115.2 54.4)
-		(end 121 54.4)
+		(start 118.5 54.5)
+		(end 121.1 54.5)
 		(width 0.4)
 		(layer "F.Cu")
@@
 	)
 	(segment
-		(start 121 54.4)
+		(start 121.1 54.5)
 		(end 122.3 55.7)
 		(width 0.4)
@@
 	(segment
 		(start 130.9 50)
-		(end 131.5 49.4)
+		(end 131.4 49.5)
 		(width 0.4)
 		(layer "F.Cu")
@@
 	)
 	(segment
-		(start 131.5 49.4)
-		(end 138.5 49.4)
+		(start 131.4 49.5)
+		(end 138.6 49.5)
 		(width 0.4)
 		(layer "F.Cu")
@@
 	)
 	(segment
-		(start 138.5 49.4)
+		(start 138.6 49.5)
 		(end 142.5 53.4)
 		(width 0.4)
@@
 		(end 114.1 59.1)
 		(width 0.4)
-		(layer "F.Cu")
+		(layer "B.Cu")
 		(net 70)
 	)
@@
 		(end 114.1 57)
 		(width 0.4)
-		(layer "F.Cu")
+		(layer "B.Cu")
 		(net 70)
 	)
@@
 		(end 114.34 56.3)
 		(width 0.4)
-		(layer "F.Cu")
+		(layer "B.Cu")
 		(net 70)
 	)
@@
 	(segment
 		(start 82.09 48.68)
-		(end 82.6 49.2)
+		(end 82.7 48.3)
 		(width 0.4)
-		(layer "F.Cu")
+		(layer "B.Cu")
 		(net 79)
 	)
 	(segment
-		(start 82.6 49.2)
-		(end 89.7 56.3)
+		(start 82.7 48.3)
+		(end 82.7 41.1)
 		(width 0.4)
-		(layer "F.Cu")
+		(layer "B.Cu")
 		(net 79)
 	)
 	(segment
-		(start 89.7 56.3)
-		(end 89.7 58.8)
+		(start 82.7 41.1)
+		(end 85.4 38.4)
 		(width 0.4)
-		(layer "F.Cu")
+		(layer "B.Cu")
 		(net 79)
 	)
 	(segment
-		(start 89.7 58.8)
-		(end 90.26 59.295)
+		(start 85.4 38.4)
+		(end 86 38.02)
 		(width 0.4)
-		(layer "F.Cu")
+		(layer "B.Cu")
 		(net 79)
 	)
 	(segment
-		(start 90.26 59.295)
-		(end 90.8 59.8)
+		(start 71.66 53.13)
+		(end 72.3 53.5)
 		(width 0.4)
-		(layer "F.Cu")
+		(layer "B.Cu")
 		(net 79)
 	)
 	(segment
-		(start 90.8 59.8)
-		(end 90.8 61.3)
+		(start 72.3 53.5)
+		(end 73.7 54.9)
 		(width 0.4)
-		(layer "F.Cu")
+		(layer "B.Cu")
 		(net 79)
 	)
 	(segment
-		(start 90.8 61.3)
-		(end 92.2 62.7)
+		(start 73.7 54.9)
+		(end 73.7 58.1)
 		(width 0.4)
-		(layer "F.Cu")
+		(layer "B.Cu")
 		(net 79)
 	)
 	(segment
-		(start 92.2 62.7)
-		(end 92.8 63.105)
+		(start 73.7 58.1)
+		(end 80.3 58.1)
 		(width 0.4)
-		(layer "F.Cu")
+		(layer "B.Cu")
 		(net 79)
 	)
 	(segment
-		(start 90.26 59.295)
-		(end 89.6 59.5)
+		(start 80.3 58.1)
+		(end 81.5 59.3)
 		(width 0.4)
-		(layer "F.Cu")
+		(layer "B.Cu")
 		(net 79)
 	)
 	(segment
-		(start 89.6 59.5)
+		(start 81.5 59.3)
+		(end 81.82 59.93)
+		(width 0.4)
+		(layer "B.Cu")
+		(net 79)
+	)
+	(segment
+		(start 81.82 59.93)
 		(end 82.4 59.5)
 		(width 0.4)
@@
 	(segment
 		(start 82.4 59.5)
-		(end 81.82 59.93)
+		(end 89.6 59.5)
 		(width 0.4)
 		(layer "F.Cu")
@@
 	)
 	(segment
-		(start 82.09 48.68)
-		(end 82.7 48.3)
+		(start 89.6 59.5)
+		(end 90.26 59.295)
 		(width 0.4)
-		(layer "B.Cu")
+		(layer "F.Cu")
 		(net 79)
 	)
 	(segment
-		(start 82.7 48.3)
-		(end 82.7 41.1)
+		(start 90.26 59.295)
+		(end 90.8 59.8)
 		(width 0.4)
-		(layer "B.Cu")
+		(layer "F.Cu")
 		(net 79)
 	)
 	(segment
-		(start 82.7 41.1)
-		(end 85.4 38.4)
+		(start 90.8 59.8)
+		(end 90.8 61.3)
 		(width 0.4)
-		(layer "B.Cu")
+		(layer "F.Cu")
 		(net 79)
 	)
 	(segment
-		(start 85.4 38.4)
-		(end 86 38.02)
+		(start 90.8 61.3)
+		(end 92.2 62.7)
 		(width 0.4)
-		(layer "B.Cu")
+		(layer "F.Cu")
+		(net 79)
+	)
+	(segment
+		(start 92.2 62.7)
+		(end 92.8 63.105)
+		(width 0.4)
+		(layer "F.Cu")
 		(net 79)
 	)
@@
 	(segment
 		(start 106 83.5)
-		(end 106.7 82.9)
+		(end 106.9 83.2)
 		(width 0.4)
 		(layer "F.Cu")
@@
 	)
 	(segment
-		(start 106.7 82.9)
-		(end 114 75.6)
+		(start 106.9 83.2)
+		(end 114.2 75.9)
 		(width 0.4)
 		(layer "F.Cu")
@@
 	)
 	(segment
-		(start 114 75.6)
+		(start 114.2 75.9)
 		(end 114.7 75.485)
 		(width 0.4)
