File: PCB/TS06-DRV/TS06-DRV-03-hv.kicad_sch (KiCad schematic)
At the start: 22 parts, among them U11 TC4420, U12 LM393

Commit message: TS06-DRV rev B: routed - round 13, 0 nets sharing, 0 unrouted; board, rules and schematic written
The route of run r3 (PYTHONHASHSEED=0, the RC block of OPTIONS.md option 3),
polished (30 nets shorter), saved in tools/mkpcb_drv_routes.json, and the board
regenerated from it: check() 0 problems, 0 cathode pads under 0.5 mm, check_mate()
clean, 1164 segments, 0 vias. TS06-DRV.kicad_dru carries the 0.8 mm HV pad rule.
Schematic regenerated by tools/mksch_pair.py; BOMs unchanged by tools/bom_pair.py.

State: board written from a converged route; verify_pair not yet run.
Blocker: none.
Next: verify_pair.sh, scorecard, README row.

Co-Authored-By: Claude Opus 5.5 <noreply@anthropic.com>
Claude-Session: https://claude.ai/code/session_01WoV3gyAFgmtuk6W6Dr4bdA
Parts:
- added R75: 100k, TS06:TS06_R_Axial_DIN0207_P10.16mm_R180, symbol TS06_pair:R
- added R76: 10k, TS06:TS06_R_Axial_DIN0207_P10.16mm, symbol TS06_pair:R
- added VD5: 1N4762A, TS06:TS06_D_DO-41_P10.16mm, symbol TS06_pair:D_Zener
- added VD6: 1N4762A, TS06:TS06_D_DO-41_P10.16mm_R180, symbol TS06_pair:D_Zener
- added VD7: 1N4761A, TS06:TS06_D_DO-41_P10.16mm, symbol TS06_pair:D_Zener
- added VT2: 2N3904, TS06:TS06_TO-92_Inline_Wide_R180, symbol TS06_pair:Q_NPN_EBC
- C12: footprint TS06:TS06_C_Disc_P5.00mm -> TS06:TS06_C_Disc_P5.00mm_R270
- C13: footprint TS06:TS06_C_Disc_P5.00mm_R90 -> TS06:TS06_C_Disc_P5.00mm_R180
- C7: footprint TS06:TS06_CP_Radial_D10.0mm_P5.00mm -> TS06:TS06_CP_Radial_D10.0mm_P5.00mm_R180
- L1: value 220u 2A -> 220u 1.8A 5900-221-RC; footprint TS06:TS06_L_Radial_D12.0mm_P5.00mm -> TS06:TS06_L_Axial_D11.5mm_L22.9mm_P27.94mm
- R60, R61, R62: footprint TS06:TS06_R_Axial_DIN0309_P12.70mm -> TS06:TS06_R_Axial_MLT-0.5_P15.24mm
- R63: footprint TS06:TS06_R_Axial_DIN0309_P12.70mm_R270 -> TS06:TS06_R_Axial_MLT-0.5_P15.24mm_R270
- R65: footprint TS06:TS06_R_Axial_DIN0207_P10.16mm -> TS06:TS06_R_Axial_DIN0207_P2.54mm_Vertical_R180
- R67: footprint TS06:TS06_R_Axial_DIN0207_P10.16mm_R180 -> TS06:TS06_R_Axial_DIN0207_P2.54mm_Vertical
- R68: footprint TS06:TS06_R_Axial_DIN0207_P10.16mm -> TS06:TS06_R_Axial_DIN0207_P2.54mm_Vertical_R90
- R69, R70: footprint TS06:TS06_R_Axial_DIN0207_P10.16mm_R90 -> TS06:TS06_R_Axial_DIN0207_P2.54mm_Vertical_R90
- R71: footprint TS06:TS06_R_Axial_DIN0207_P10.16mm_R90 -> TS06:TS06_R_Axial_DIN0207_P2.54mm_Vertical_R180
- U11: footprint TS06:TS06_DIP-8_W7.62mm_Socket_R180 -> TS06:TS06_DIP-8_W7.62mm_Socket
Connections:
- net GND: now also R76.2, VT2.1 (E)
- net HV185: now also VD5.1 (K)
- net PWM_G: now also VT2.3 (C)
- new net OVZ_1: VD5.2 (A), VD6.1 (K)
- new net OVZ_2: VD6.2 (A), VD7.1 (K)
- new net OVZ_3: R75.1, VD7.2 (A)
- new net OV_B: R75.2, R76.1, VT2.2 (B)
Other:
- note added: "C7: The reservoir, 400 V. L1: Bourns 5900-221-RC: 220 uH, Isat 1.8 A, Irated 1.6 A, DCR 0.162 ohm; axial, lying, 1.1 mm holes 27.94 mm apart. R60: Bleeder: the reservoir is safe ~10 s after power-off. R62: Divider top, two in series: ~92 V each at 185 V and ~104 V at the trimmer's 210 V end, against the part's 350 V rating. R65: Hysteresis, about 1 V of rail. R67: Standing, between the driver's o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"
- note added: "Parts this sheet's layout does not know yet (added to tools/ts06pair.py since): labelled, not wired."
- note removed: "C7: The reservoir, 400 V. L1: 220 uH, Isat >= 1.8 A (1.3 A peaks at 12 V in, 23.8 us on). R60: Bleeder: the reservoir is safe ~10 s after power-off. R62: Divider top, two in series, each under 100 V. R65: Hysteresis, about 1 V of rail. R69: 2.5 V reference. RP1: Rail set-point 165-210 V; wiper on the grounded end, so an open wiper lowers the rail. U11: Non-inverting MOSFET driver, 12 V out. MCP14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"
