File: PCB/TS06-DRV/TS06-DRV-05-decoders.kicad_sch (KiCad schematic)
At the start: 4 parts, among them U17 K155ID1, U2 K155ID1

Commit message: TS06-DRV rev B: routed - round 13, 0 nets sharing, 0 unrouted; board, rules and schematic written
The route of run r3 (PYTHONHASHSEED=0, the RC block of OPTIONS.md option 3),
polished (30 nets shorter), saved in tools/mkpcb_drv_routes.json, and the board
regenerated from it: check() 0 problems, 0 cathode pads under 0.5 mm, check_mate()
clean, 1164 segments, 0 vias. TS06-DRV.kicad_dru carries the 0.8 mm HV pad rule.
Schematic regenerated by tools/mksch_pair.py; BOMs unchanged by tools/bom_pair.py.

State: board written from a converged route; verify_pair not yet run.
Blocker: none.
Next: verify_pair.sh, scorecard, README row.

Co-Authored-By: Claude Opus 5.5 <noreply@anthropic.com>
Claude-Session: https://claude.ai/code/session_01WoV3gyAFgmtuk6W6Dr4bdA
Parts:
- U17: footprint TS06:TS06_DIP-16_W7.62mm_Socket_R90 -> TS06:TS06_DIP-16_W7.62mm_Socket_Oval_R90
- U2: footprint TS06:TS06_DIP-16_W7.62mm_Socket_R180 -> TS06:TS06_DIP-16_W7.62mm_Socket_Oval_R180
Changed lines of the file:
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@@
 )
 )
-(property "Footprint" "TS06:TS06_DIP-16_W7.62mm_Socket_R180"
+(property "Footprint" "TS06:TS06_DIP-16_W7.62mm_Socket_Oval_R180"
 (at 88.9 45.72 0)
 (hide yes)
@@
 )
 )
-(property "Footprint" "TS06:TS06_DIP-16_W7.62mm_Socket_R90"
+(property "Footprint" "TS06:TS06_DIP-16_W7.62mm_Socket_Oval_R90"
 (at 203.2 45.72 0)
 (hide yes)
@@
 (on_board yes)
 (dnp no)
-(property "Reference" "#PWR038"
+(property "Reference" "#PWR043"
 (at 76.2 46.99 0)
 (hide yes)
@@
 (project "TS06-DRV"
 (path "/581aa1b9-f775-5fe0-87f7-a79eaeda6019/d8e7b9af-4d19-586f-ae83-3ca65b61d572"
-(reference "#PWR038")
+(reference "#PWR043")
 (unit 1)
 )
@@
 (on_board yes)
 (dnp no)
-(property "Reference" "#PWR039"
+(property "Reference" "#PWR044"
 (at 88.9 66.04 0)
 (hide yes)
@@
 (project "TS06-DRV"
 (path "/581aa1b9-f775-5fe0-87f7-a79eaeda6019/d8e7b9af-4d19-586f-ae83-3ca65b61d572"
-(reference "#PWR039")
+(reference "#PWR044")
 (unit 1)
 )
@@
 (on_board yes)
 (dnp no)
-(property "Reference" "#PWR040"
+(property "Reference" "#PWR045"
 (at 190.5 46.99 0)
 (hide yes)
@@
 (project "TS06-DRV"
 (path "/581aa1b9-f775-5fe0-87f7-a79eaeda6019/d8e7b9af-4d19-586f-ae83-3ca65b61d572"
-(reference "#PWR040")
+(reference "#PWR045")
 (unit 1)
 )
@@
 (on_board yes)
 (dnp no)
-(property "Reference" "#PWR041"
+(property "Reference" "#PWR046"
 (at 203.2 66.04 0)
 (hide yes)
@@
 (project "TS06-DRV"
 (path "/581aa1b9-f775-5fe0-87f7-a79eaeda6019/d8e7b9af-4d19-586f-ae83-3ca65b61d572"
-(reference "#PWR041")
+(reference "#PWR046")
 (unit 1)
 )
@@
 (on_board yes)
 (dnp no)
-(property "Reference" "#PWR042"
+(property "Reference" "#PWR047"
 (at 88.9 78.74 0)
 (hide yes)
@@
 (project "TS06-DRV"
 (path "/581aa1b9-f775-5fe0-87f7-a79eaeda6019/d8e7b9af-4d19-586f-ae83-3ca65b61d572"
-(reference "#PWR042")
+(reference "#PWR047")
 (unit 1)
 )
@@
 (on_board yes)
 (dnp no)
-(property "Reference" "#PWR043"
+(property "Reference" "#PWR048"
 (at 101.6 46.99 0)
 (hide yes)
@@
 (project "TS06-DRV"
 (path "/581aa1b9-f775-5fe0-87f7-a79eaeda6019/d8e7b9af-4d19-586f-ae83-3ca65b61d572"
-(reference "#PWR043")
+(reference "#PWR048")
 (unit 1)
 )
@@
 (on_board yes)
 (dnp no)
-(property "Reference" "#PWR044"
+(property "Reference" "#PWR049"
 (at 203.2 78.74 0)
 (hide yes)
@@
 (project "TS06-DRV"
 (path "/581aa1b9-f775-5fe0-87f7-a79eaeda6019/d8e7b9af-4d19-586f-ae83-3ca65b61d572"
-(reference "#PWR044")
+(reference "#PWR049")
 (unit 1)
 )
@@
 (on_board yes)
 (dnp no)
-(property "Reference" "#PWR045"
+(property "Reference" "#PWR050"
 (at 215.9 46.99 0)
 (hide yes)
@@
 (project "TS06-DRV"
 (path "/581aa1b9-f775-5fe0-87f7-a79eaeda6019/d8e7b9af-4d19-586f-ae83-3ca65b61d572"
-(reference "#PWR045")
-(unit 1)
-)
+(reference "#PWR050")
+(unit 1)
+)
