File: PCB/TS06-DRV/TS06-DRV-06-anodes.kicad_sch (KiCad schematic)
At the start: 30 parts, among them U10 TLP627, U5 TLP627, U6 TLP627, U7 TLP627, U8 TLP627, U9 TLP627

Commit message: TS06-DRV rev B: routed - round 13, 0 nets sharing, 0 unrouted; board, rules and schematic written
The route of run r3 (PYTHONHASHSEED=0, the RC block of OPTIONS.md option 3),
polished (30 nets shorter), saved in tools/mkpcb_drv_routes.json, and the board
regenerated from it: check() 0 problems, 0 cathode pads under 0.5 mm, check_mate()
clean, 1164 segments, 0 vias. TS06-DRV.kicad_dru carries the 0.8 mm HV pad rule.
Schematic regenerated by tools/mksch_pair.py; BOMs unchanged by tools/bom_pair.py.

State: board written from a converged route; verify_pair not yet run.
Blocker: none.
Next: verify_pair.sh, scorecard, README row.

Co-Authored-By: Claude Opus 5.5 <noreply@anthropic.com>
Claude-Session: https://claude.ai/code/session_01WoV3gyAFgmtuk6W6Dr4bdA
Parts:
- R27, R28, R32: footprint TS06:TS06_R_Axial_DIN0309_P12.70mm -> TS06:TS06_R_Axial_MLT-0.5_P15.24mm
- R29, R30: footprint TS06:TS06_R_Axial_DIN0309_P12.70mm_R180 -> TS06:TS06_R_Axial_MLT-0.5_P15.24mm
- R31: footprint TS06:TS06_R_Axial_DIN0309_P12.70mm -> TS06:TS06_R_Axial_MLT-0.5_P15.24mm_R180
- R33, R34, R35, R36, R42, R43: now not fitted
- R37, R38, R39: footprint TS06:TS06_R_Axial_DIN0207_P2.54mm_Vertical_R180 -> TS06:TS06_R_Axial_DIN0207_P2.54mm_Vertical; now not fitted
- R40: footprint TS06:TS06_R_Axial_DIN0207_P2.54mm_Vertical_R90 -> TS06:TS06_R_Axial_DIN0207_P2.54mm_Vertical; now not fitted
- R41, R44: footprint TS06:TS06_R_Axial_DIN0207_P2.54mm_Vertical -> TS06:TS06_R_Axial_DIN0207_P2.54mm_Vertical_R90; now not fitted
Changed lines of the file:
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@@
 )
 )
-(property "Footprint" "TS06:TS06_R_Axial_DIN0309_P12.70mm"
+(property "Footprint" "TS06:TS06_R_Axial_MLT-0.5_P15.24mm"
 (at 69.85 50.8 0)
 (hide yes)
@@
 )
 )
-(property "Footprint" "TS06:TS06_R_Axial_DIN0309_P12.70mm"
+(property "Footprint" "TS06:TS06_R_Axial_MLT-0.5_P15.24mm"
 (at 196.85 50.8 0)
 (hide yes)
@@
 )
 )
-(property "Footprint" "TS06:TS06_R_Axial_DIN0309_P12.70mm_R180"
+(property "Footprint" "TS06:TS06_R_Axial_MLT-0.5_P15.24mm"
 (at 323.85 50.8 0)
 (hide yes)
@@
 )
 )
-(property "Footprint" "TS06:TS06_R_Axial_DIN0309_P12.70mm_R180"
+(property "Footprint" "TS06:TS06_R_Axial_MLT-0.5_P15.24mm"
 (at 69.85 109.22 0)
 (hide yes)
@@
 )
 )
-(property "Footprint" "TS06:TS06_R_Axial_DIN0309_P12.70mm"
+(property "Footprint" "TS06:TS06_R_Axial_MLT-0.5_P15.24mm_R180"
 (at 196.85 109.22 0)
 (hide yes)
@@
 )
 )
-(property "Footprint" "TS06:TS06_R_Axial_DIN0309_P12.70mm"
+(property "Footprint" "TS06:TS06_R_Axial_MLT-0.5_P15.24mm"
 (at 323.85 109.22 0)
 (hide yes)
@@
 (on_board yes)
 (in_pos_files yes)
-(dnp no)
+(dnp yes)
 (property "Reference" "R33"
 (at 85.09 62.23 0)
@@
 (on_board yes)
 (in_pos_files yes)
-(dnp no)
+(dnp yes)
 (property "Reference" "R34"
 (at 85.09 72.39 0)
@@
 (on_board yes)
 (in_pos_files yes)
-(dnp no)
+(dnp yes)
 (property "Reference" "R35"
 (at 212.09 62.23 0)
@@
 (on_board yes)
 (in_pos_files yes)
-(dnp no)
+(dnp yes)
 (property "Reference" "R36"
 (at 212.09 72.39 0)
@@
 (on_board yes)
 (in_pos_files yes)
-(dnp no)
+(dnp yes)
 (property "Reference" "R37"
 (at 339.09 62.23 0)
@@
 )
 )
-(property "Footprint" "TS06:TS06_R_Axial_DIN0207_P2.54mm_Vertical_R180"
+(property "Footprint" "TS06:TS06_R_Axial_DIN0207_P2.54mm_Vertical"
 (at 336.55 63.5 0)
 (hide yes)
@@
 (on_board yes)
 (in_pos_files yes)
-(dnp no)
+(dnp yes)
 (property "Reference" "R38"
 (at 339.09 72.39 0)
@@
 )
 )
-(property "Footprint" "TS06:TS06_R_Axial_DIN0207_P2.54mm_Vertical_R180"
+(property "Footprint" "TS06:TS06_R_Axial_DIN0207_P2.54mm_Vertical"
 (at 336.55 73.66 0)
 (hide yes)
@@
 (on_board yes)
 (in_pos_files yes)
-(dnp no)
+(dnp yes)
 (property "Reference" "R39"
 (at 85.09 120.65 0)
@@
 )
 )
-(property "Footprint" "TS06:TS06_R_Axial_DIN0207_P2.54mm_Vertical_R180"
+(property "Footprint" "TS06:TS06_R_Axial_DIN0207_P2.54mm_Vertical"
 (at 82.55 121.92 0)
 (hide yes)
@@
 (on_board yes)
 (in_pos_files yes)
-(dnp no)
+(dnp yes)
 (property "Reference" "R40"
 (at 85.09 130.81 0)
@@
 )
 )
-(property "Footprint" "TS06:TS06_R_Axial_DIN0207_P2.54mm_Vertical_R90"
+(property "Footprint" "TS06:TS06_R_Axial_DIN0207_P2.54mm_Vertical"
 (at 82.55 132.08 0)
 (hide yes)
@@
 (on_board yes)
 (in_pos_files yes)
-(dnp no)
+(dnp yes)
 (property "Reference" "R41"
 (at 212.09 120.65 0)
@@
 )
 )
-(property "Footprint" "TS06:TS06_R_Axial_DIN0207_P2.54mm_Vertical"
+(property "Footprint" "TS06:TS06_R_Axial_DIN0207_P2.54mm_Vertical_R90"
 (at 209.55 121.92 0)
 (hide yes)
@@
 (on_board yes)
 (in_pos_files yes)
-(dnp no)
+(dnp yes)
 (property "Reference" "R42"
 (at 212.09 130.81 0)
@@
 (on_board yes)
 (in_pos_files yes)
-(dnp no)
+(dnp yes)
 (property "Reference" "R43"
 (at 339.09 120.65 0)
@@
 (on_board yes)
 (in_pos_files yes)
-(dnp no)
+(dnp yes)
 (property "Reference" "R44"
 (at 339.09 130.81 0)
@@
 )
 )
-(property "Footprint" "TS06:TS06_R_Axial_DIN0207_P2.54mm_Vertical"
+(property "Footprint" "TS06:TS06_R_Axial_DIN0207_P2.54mm_Vertical_R90"
 (at 336.55 132.08 0)
 (hide yes)
@@
 (on_board yes)
 (dnp no)
-(property "Reference" "#PWR046"
+(property "Reference" "#PWR051"
 (at 41.91 43.18 0)
 (hide yes)
@@
 (project "TS06-DRV"
 (path "/581aa1b9-f775-5fe0-87f7-a79eaeda6019/f440e997-3d91-59c8-8109-dd8fb6052483"
-(reference "#PWR046")
+(reference "#PWR051")
 (unit 1)
 )
@@
 (on_board yes)
 (dnp no)
-(property "Reference" "#PWR047"
+(property "Reference" "#PWR052"
 (at 41.91 101.6 0)
 (hide yes)
@@
 (project "TS06-DRV"
 (path "/581aa1b9-f775-5fe0-87f7-a79eaeda6019/f440e997-3d91-59c8-8109-dd8fb6052483"
-(reference "#PWR047")
+(reference "#PWR052")
 (unit 1)
 )
@@
 (on_board yes)
 (dnp no)
-(property "Reference" "#PWR048"
+(property "Reference" "#PWR053"
 (at 82.55 80.01 0)
 (hide yes)
@@
 (project "TS06-DRV"
 (path "/581aa1b9-f775-5fe0-87f7-a79eaeda6019/f440e997-3d91-59c8-8109-dd8fb6052483"
-(reference "#PWR048")
+(reference "#PWR053")
 (unit 1)
 )
@@
 (on_board yes)
 (dnp no)
-(property "Reference" "#PWR049"
+(property "Reference" "#PWR054"
 (at 82.55 138.43 0)
 (hide yes)
@@
 (project "TS06-DRV"
 (path "/581aa1b9-f775-5fe0-87f7-a79eaeda6019/f440e997-3d91-59c8-8109-dd8fb6052483"
-(reference "#PWR049")
+(reference "#PWR054")
 (unit 1)
 )
@@
 (on_board yes)
 (dnp no)
-(property "Reference" "#PWR050"
+(property "Reference" "#PWR055"
 (at 168.91 43.18 0)
 (hide yes)
@@
 (project "TS06-DRV"
 (path "/581aa1b9-f775-5fe0-87f7-a79eaeda6019/f440e997-3d91-59c8-8109-dd8fb6052483"
-(reference "#PWR050")
+(reference "#PWR055")
 (unit 1)
 )
@@
 (on_board yes)
 (dnp no)
-(property "Reference" "#PWR051"
+(property "Reference" "#PWR056"
 (at 168.91 101.6 0)
 (hide yes)
@@
 (project "TS06-DRV"
 (path "/581aa1b9-f775-5fe0-87f7-a79eaeda6019/f440e997-3d91-59c8-8109-dd8fb6052483"
-(reference "#PWR051")
+(reference "#PWR056")
 (unit 1)
 )
@@
 (on_board yes)
 (dnp no)
-(property "Reference" "#PWR052"
+(property "Reference" "#PWR057"
 (at 209.55 80.01 0)
 (hide yes)
@@
 (project "TS06-DRV"
 (path "/581aa1b9-f775-5fe0-87f7-a79eaeda6019/f440e997-3d91-59c8-8109-dd8fb6052483"
-(reference "#PWR052")
+(reference "#PWR057")
 (unit 1)
 )
@@
 (on_board yes)
 (dnp no)
-(property "Reference" "#PWR053"
+(property "Reference" "#PWR058"
 (at 209.55 138.43 0)
 (hide yes)
@@
 (project "TS06-DRV"
 (path "/581aa1b9-f775-5fe0-87f7-a79eaeda6019/f440e997-3d91-59c8-8109-dd8fb6052483"
-(reference "#PWR053")
+(reference "#PWR058")
 (unit 1)
 )
@@
 (on_board yes)
 (dnp no)
-(property "Reference" "#PWR054"
+(property "Reference" "#PWR059"
 (at 295.91 43.18 0)
 (hide yes)
@@
 (project "TS06-DRV"
 (path "/581aa1b9-f775-5fe0-87f7-a79eaeda6019/f440e997-3d91-59c8-8109-dd8fb6052483"
-(reference "#PWR054")
+(reference "#PWR059")
 (unit 1)
 )
@@
 (on_board yes)
 (dnp no)
-(property "Reference" "#PWR055"
+(property "Reference" "#PWR060"
 (at 295.91 101.6 0)
 (hide yes)
@@
 (project "TS06-DRV"
 (path "/581aa1b9-f775-5fe0-87f7-a79eaeda6019/f440e997-3d91-59c8-8109-dd8fb6052483"
-(reference "#PWR055")
+(reference "#PWR060")
 (unit 1)
 )
@@
 (on_board yes)
 (dnp no)
-(property "Reference" "#PWR056"
+(property "Reference" "#PWR061"
 (at 336.55 80.01 0)
 (hide yes)
@@
 (project "TS06-DRV"
 (path "/581aa1b9-f775-5fe0-87f7-a79eaeda6019/f440e997-3d91-59c8-8109-dd8fb6052483"
-(reference "#PWR056")
+(reference "#PWR061")
 (unit 1)
 )
@@
 (on_board yes)
 (dnp no)
-(property "Reference" "#PWR057"
+(property "Reference" "#PWR062"
 (at 336.55 138.43 0)
 (hide yes)
@@
 (project "TS06-DRV"
 (path "/581aa1b9-f775-5fe0-87f7-a79eaeda6019/f440e997-3d91-59c8-8109-dd8fb6052483"
-(reference "#PWR057")
-(unit 1)
-)
+(reference "#PWR062")
+(unit 1)
+)
