File: PCB/TS06-DRV/TS06-DRV-07-colon.kicad_sch (KiCad schematic)
At the start: 4 parts

Commit message: TS06-DRV rev B: routed - round 13, 0 nets sharing, 0 unrouted; board, rules and schematic written
The route of run r3 (PYTHONHASHSEED=0, the RC block of OPTIONS.md option 3),
polished (30 nets shorter), saved in tools/mkpcb_drv_routes.json, and the board
regenerated from it: check() 0 problems, 0 cathode pads under 0.5 mm, check_mate()
clean, 1164 segments, 0 vias. TS06-DRV.kicad_dru carries the 0.8 mm HV pad rule.
Schematic regenerated by tools/mksch_pair.py; BOMs unchanged by tools/bom_pair.py.

State: board written from a converged route; verify_pair not yet run.
Blocker: none.
Next: verify_pair.sh, scorecard, README row.

Co-Authored-By: Claude Opus 5.5 <noreply@anthropic.com>
Claude-Session: https://claude.ai/code/session_01WoV3gyAFgmtuk6W6Dr4bdA
Parts:
- R58, R59: footprint TS06:TS06_R_Axial_DIN0309_P12.70mm_R270 -> TS06:TS06_R_Axial_MLT-0.5_P15.24mm_R270
Changed lines of the file:
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@@
 )
 )
-(property "Footprint" "TS06:TS06_R_Axial_DIN0309_P12.70mm_R270"
+(property "Footprint" "TS06:TS06_R_Axial_MLT-0.5_P15.24mm_R270"
 (at 59.69 35.56 0)
 (hide yes)
@@
 )
 )
-(property "Footprint" "TS06:TS06_R_Axial_DIN0309_P12.70mm_R270"
+(property "Footprint" "TS06:TS06_R_Axial_MLT-0.5_P15.24mm_R270"
 (at 59.69 45.72 0)
 (hide yes)
@@
 (on_board yes)
 (dnp no)
-(property "Reference" "#PWR058"
+(property "Reference" "#PWR063"
 (at 76.2 78.74 0)
 (hide yes)
@@
 (project "TS06-DRV"
 (path "/581aa1b9-f775-5fe0-87f7-a79eaeda6019/9a1a64a8-3db4-522f-a34c-c12ebb816af2"
-(reference "#PWR058")
-(unit 1)
-)
+(reference "#PWR063")
+(unit 1)
+)
