File: PCB/TS06-DRV/TS06-DRV-08-ampm.kicad_sch (KiCad schematic)
At the start: 8 parts, among them U15 K155ID1, U16 K155ID1, U3 MCP23017-E/SP

Commit message: TS06-DRV rev B: routed - round 13, 0 nets sharing, 0 unrouted; board, rules and schematic written
The route of run r3 (PYTHONHASHSEED=0, the RC block of OPTIONS.md option 3),
polished (30 nets shorter), saved in tools/mkpcb_drv_routes.json, and the board
regenerated from it: check() 0 problems, 0 cathode pads under 0.5 mm, check_mate()
clean, 1164 segments, 0 vias. TS06-DRV.kicad_dru carries the 0.8 mm HV pad rule.
Schematic regenerated by tools/mksch_pair.py; BOMs unchanged by tools/bom_pair.py.

State: board written from a converged route; verify_pair not yet run.
Blocker: none.
Next: verify_pair.sh, scorecard, README row.

Co-Authored-By: Claude Opus 5.5 <noreply@anthropic.com>
Claude-Session: https://claude.ai/code/session_01WoV3gyAFgmtuk6W6Dr4bdA
Parts:
- R56, R57: footprint TS06:TS06_R_Axial_DIN0309_P12.70mm_R180 -> TS06:TS06_R_Axial_MLT-0.5_P15.24mm
- U15, U16: footprint TS06:TS06_DIP-16_W7.62mm_Socket_R90 -> TS06:TS06_DIP-16_W7.62mm_Socket_Oval_R90
Changed lines of the file:
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@@
 )
 )
-(property "Footprint" "TS06:TS06_R_Axial_DIN0309_P12.70mm_R180"
+(property "Footprint" "TS06:TS06_R_Axial_MLT-0.5_P15.24mm"
 (at 283.21 35.56 0)
 (hide yes)
@@
 )
 )
-(property "Footprint" "TS06:TS06_R_Axial_DIN0309_P12.70mm_R180"
+(property "Footprint" "TS06:TS06_R_Axial_MLT-0.5_P15.24mm"
 (at 283.21 45.72 0)
 (hide yes)
@@
 )
 )
-(property "Footprint" "TS06:TS06_DIP-16_W7.62mm_Socket_R90"
+(property "Footprint" "TS06:TS06_DIP-16_W7.62mm_Socket_Oval_R90"
 (at 177.8 106.68 0)
 (hide yes)
@@
 )
 )
-(property "Footprint" "TS06:TS06_DIP-16_W7.62mm_Socket_R90"
+(property "Footprint" "TS06:TS06_DIP-16_W7.62mm_Socket_Oval_R90"
 (at 177.8 71.12 0)
 (hide yes)
@@
 (on_board yes)
 (dnp no)
-(property "Reference" "#PWR059"
+(property "Reference" "#PWR064"
 (at 60.96 85.09 0)
 (hide yes)
@@
 (project "TS06-DRV"
 (path "/581aa1b9-f775-5fe0-87f7-a79eaeda6019/aea59eb5-c86f-5aa6-b1f8-4218445b4b15"
-(reference "#PWR059")
+(reference "#PWR064")
 (unit 1)
 )
@@
 (on_board yes)
 (dnp no)
-(property "Reference" "#PWR060"
+(property "Reference" "#PWR065"
 (at 76.2 109.22 0)
 (hide yes)
@@
 (project "TS06-DRV"
 (path "/581aa1b9-f775-5fe0-87f7-a79eaeda6019/aea59eb5-c86f-5aa6-b1f8-4218445b4b15"
-(reference "#PWR060")
+(reference "#PWR065")
 (unit 1)
 )
@@
 (on_board yes)
 (dnp no)
-(property "Reference" "#PWR061"
+(property "Reference" "#PWR066"
 (at 91.44 90.17 0)
 (hide yes)
@@
 (project "TS06-DRV"
 (path "/581aa1b9-f775-5fe0-87f7-a79eaeda6019/aea59eb5-c86f-5aa6-b1f8-4218445b4b15"
-(reference "#PWR061")
+(reference "#PWR066")
 (unit 1)
 )
@@
 (on_board yes)
 (dnp no)
-(property "Reference" "#PWR062"
+(property "Reference" "#PWR067"
 (at 165.1 72.39 0)
 (hide yes)
@@
 (project "TS06-DRV"
 (path "/581aa1b9-f775-5fe0-87f7-a79eaeda6019/aea59eb5-c86f-5aa6-b1f8-4218445b4b15"
-(reference "#PWR062")
+(reference "#PWR067")
 (unit 1)
 )
@@
 (on_board yes)
 (dnp no)
-(property "Reference" "#PWR063"
+(property "Reference" "#PWR068"
 (at 165.1 107.95 0)
 (hide yes)
@@
 (project "TS06-DRV"
 (path "/581aa1b9-f775-5fe0-87f7-a79eaeda6019/aea59eb5-c86f-5aa6-b1f8-4218445b4b15"
-(reference "#PWR063")
+(reference "#PWR068")
 (unit 1)
 )
@@
 (on_board yes)
 (dnp no)
-(property "Reference" "#PWR064"
+(property "Reference" "#PWR069"
 (at 223.52 62.23 0)
 (hide yes)
@@
 (project "TS06-DRV"
 (path "/581aa1b9-f775-5fe0-87f7-a79eaeda6019/aea59eb5-c86f-5aa6-b1f8-4218445b4b15"
-(reference "#PWR064")
+(reference "#PWR069")
 (unit 1)
 )
@@
 (on_board yes)
 (dnp no)
-(property "Reference" "#PWR065"
+(property "Reference" "#PWR070"
 (at 223.52 97.79 0)
 (hide yes)
@@
 (project "TS06-DRV"
 (path "/581aa1b9-f775-5fe0-87f7-a79eaeda6019/aea59eb5-c86f-5aa6-b1f8-4218445b4b15"
-(reference "#PWR065")
+(reference "#PWR070")
 (unit 1)
 )
@@
 (on_board yes)
 (dnp no)
-(property "Reference" "#PWR066"
+(property "Reference" "#PWR071"
 (at 60.96 87.63 0)
 (hide yes)
@@
 (project "TS06-DRV"
 (path "/581aa1b9-f775-5fe0-87f7-a79eaeda6019/aea59eb5-c86f-5aa6-b1f8-4218445b4b15"
-(reference "#PWR066")
+(reference "#PWR071")
 (unit 1)
 )
@@
 (on_board yes)
 (dnp no)
-(property "Reference" "#PWR067"
+(property "Reference" "#PWR072"
 (at 76.2 121.92 0)
 (hide yes)
@@
 (project "TS06-DRV"
 (path "/581aa1b9-f775-5fe0-87f7-a79eaeda6019/aea59eb5-c86f-5aa6-b1f8-4218445b4b15"
-(reference "#PWR067")
+(reference "#PWR072")
 (unit 1)
 )
@@
 (on_board yes)
 (dnp no)
-(property "Reference" "#PWR068"
+(property "Reference" "#PWR073"
 (at 91.44 100.33 0)
 (hide yes)
@@
 (project "TS06-DRV"
 (path "/581aa1b9-f775-5fe0-87f7-a79eaeda6019/aea59eb5-c86f-5aa6-b1f8-4218445b4b15"
-(reference "#PWR068")
+(reference "#PWR073")
 (unit 1)
 )
@@
 (on_board yes)
 (dnp no)
-(property "Reference" "#PWR069"
+(property "Reference" "#PWR074"
 (at 190.5 72.39 0)
 (hide yes)
@@
 (project "TS06-DRV"
 (path "/581aa1b9-f775-5fe0-87f7-a79eaeda6019/aea59eb5-c86f-5aa6-b1f8-4218445b4b15"
-(reference "#PWR069")
+(reference "#PWR074")
 (unit 1)
 )
@@
 (on_board yes)
 (dnp no)
-(property "Reference" "#PWR070"
+(property "Reference" "#PWR075"
 (at 190.5 107.95 0)
 (hide yes)
@@
 (project "TS06-DRV"
 (path "/581aa1b9-f775-5fe0-87f7-a79eaeda6019/aea59eb5-c86f-5aa6-b1f8-4218445b4b15"
-(reference "#PWR070")
+(reference "#PWR075")
 (unit 1)
 )
@@
 (on_board yes)
 (dnp no)
-(property "Reference" "#PWR071"
+(property "Reference" "#PWR076"
 (at 223.52 74.93 0)
 (hide yes)
@@
 (project "TS06-DRV"
 (path "/581aa1b9-f775-5fe0-87f7-a79eaeda6019/aea59eb5-c86f-5aa6-b1f8-4218445b4b15"
-(reference "#PWR071")
+(reference "#PWR076")
 (unit 1)
 )
@@
 (on_board yes)
 (dnp no)
-(property "Reference" "#PWR072"
+(property "Reference" "#PWR077"
 (at 223.52 110.49 0)
 (hide yes)
@@
 (project "TS06-DRV"
 (path "/581aa1b9-f775-5fe0-87f7-a79eaeda6019/aea59eb5-c86f-5aa6-b1f8-4218445b4b15"
-(reference "#PWR072")
-(unit 1)
-)
+(reference "#PWR077")
+(unit 1)
+)
