File: PCB/TS06-DRV/TS06-DRV.kicad_pcb (KiCad board)
At the start: 2 copper layers, 191.4 x 100 mm, 116 parts, among them J1 PH 6 vertical, U1 Arduino Nano, U10 TLP627, U11 TC4420, U12 LM393, U13 DS3231 mini, U14 R-78E5.0-1.0, U15 K155ID1, U16 K155ID1, U17 K155ID1, U2 K155ID1, U3 MCP23017-E/SP, U5 TLP627, U6 TLP627, U7 TLP627, U8 TLP627, U9 TLP627

Commit message: TS06-DRV rev B: J1's pinout on the display-side face reads in the order the pins stand there
Seen from the face towards the display (KiCad's mirrored plot), J1's pin 1 is on the
right; the legend read 1 to 6 from the left. It now reads 6 D8 ... 1 +5V. DRC: 0
errors, the 2 accepted Nano warnings.

State: routed, DRC clean, silk checked in KiCad's own plot (front and back).
Blocker: none in scope; 3d/case-pair outputs stale for their owner.
Next: r5 (a fresh --route, seed pinned by the script) to show the route reproduces.

Co-Authored-By: Claude Opus 5.5 <noreply@anthropic.com>
Claude-Session: https://claude.ai/code/session_01WoV3gyAFgmtuk6W6Dr4bdA
Other:
- board text added: "6 D8 5 D7 4 A7 3 A6 2 GND 1 +5V"
- board text removed: "1 +5V 2 GND 3 A6 4 A7 5 D7 6 D8"
Changed lines of the file:
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@@
 		)
 	)
-	(gr_text "1 +5V 2 GND 3 A6 4 A7 5 D7 6 D8"
+	(gr_text "6 D8 5 D7 4 A7 3 A6 2 GND 1 +5V"
 		(at 141.4 91 0)
 		(layer "B.SilkS")
