File: PCB/TS06-DRV/TS06-DRV-11-fascia.kicad_sch (KiCad schematic)
At the start: 3 parts, among them J1 PH 6 vertical

Commit message: TS06-DRV rev B: routed - round 13, 0 nets sharing, 0 unrouted; board, rules and schematic written
The route of run r3 (PYTHONHASHSEED=0, the RC block of OPTIONS.md option 3),
polished (30 nets shorter), saved in tools/mkpcb_drv_routes.json, and the board
regenerated from it: check() 0 problems, 0 cathode pads under 0.5 mm, check_mate()
clean, 1164 segments, 0 vias. TS06-DRV.kicad_dru carries the 0.8 mm HV pad rule.
Schematic regenerated by tools/mksch_pair.py; BOMs unchanged by tools/bom_pair.py.

State: board written from a converged route; verify_pair not yet run.
Blocker: none.
Next: verify_pair.sh, scorecard, README row.

Co-Authored-By: Claude Opus 5.5 <noreply@anthropic.com>
Claude-Session: https://claude.ai/code/session_01WoV3gyAFgmtuk6W6Dr4bdA
Parts:
- added C18, C19: 10n, TS06:TS06_C_Disc_P2.50mm_R270, symbol TS06_pair:C
- added R72: 1M, TS06:TS06_R_Axial_DIN0207_P10.16mm_R180, symbol TS06_pair:R
- added R73, R74: 1k, TS06:TS06_R_Axial_DIN0207_P10.16mm_R180, symbol TS06_pair:R
Connections:
- net A6: now also R72.1
- net D7: now also R73.1; no longer J1.5
- net D8: now also R74.1; no longer J1.6
- net GND: now also C18.2, C19.2, R72.2
- new net D7_J: C18.1, J1.5, R73.2
- new net D8_J: C19.1, J1.6, R74.2
Other:
- note added: "C5: Ladder filters at the board end (spec §2). C18: At J1, on the cable side of R73. J1: The panel cable; pin order is the specification both fascia builds share. Top entry, so the cable leaves towards the fascia. R72: A6 pull-down: a defined 0 with the fascia unplugged. R73: Series resistor on the button line, at J1."
- note added: "Parts this sheet's layout does not know yet (added to tools/ts06pair.py since): labelled, not wired."
- note removed: "C5: Ladder filters at the board end (spec §2). J1: The panel cable; pin order is the specification both fascia builds share. Top entry, so the cable leaves towards the fascia."

Commit message: TS06-DRV rev B: the RC parts' notes say where they now stand (between the strips and J1)
Netlist notes and the generator's docstring only; the fascia sheet regenerated by
mksch_pair.py. Board and BOM unchanged.

State: routed, DRC clean, verify 26/1 (3d/ outputs).
Blocker: none in scope.
Next: r5 reproduction; final verify; report.

Co-Authored-By: Claude Opus 5.5 <noreply@anthropic.com>
Claude-Session: https://claude.ai/code/session_01WoV3gyAFgmtuk6W6Dr4bdA
Other:
- note added: "C5: Ladder filters at the board end (spec §2). C18: Near J1, on the cable side of R73. J1: The panel cable; pin order is the specification both fascia builds share. Top entry, so the cable leaves towards the fascia. R72: A6 pull-down: a defined 0 with the fascia unplugged. R73: Series resistor on the button line, between the strips and J1."
- note removed: "C5: Ladder filters at the board end (spec §2). C18: At J1, on the cable side of R73. J1: The panel cable; pin order is the specification both fascia builds share. Top entry, so the cable leaves towards the fascia. R72: A6 pull-down: a defined 0 with the fascia unplugged. R73: Series resistor on the button line, at J1."
Changed lines of the file:
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@@
 )
 )
-(text "C5: Ladder filters at the board end (spec §2).\nC18: At J1, on the cable side of R73.\nJ1: The panel cable; pin order is the specification both fascia builds share. Top entry, so the cable leaves\ntowards the fascia.\nR72: A6 pull-down: a defined 0 with the fascia unplugged.\nR73: Series resistor on the button line, at J1."
+(text "C5: Ladder filters at the board end (spec §2).\nC18: Near J1, on the cable side of R73.\nJ1: The panel cable; pin order is the specification both fascia builds share. Top entry, so the cable leaves\ntowards the fascia.\nR72: A6 pull-down: a defined 0 with the fascia unplugged.\nR73: Series resistor on the button line, between the strips and J1."
 (exclude_from_sim no)
 (at 20.32 115.57 0)
