File: PCB/TS06-FASCIA-rhythm/TS06-FASCIA-rhythm.kicad_pcb (KiCad board)
At the start: 2 copper layers, 191.4 x 40 mm, 18 parts, among them J1 PH 6, SW1 SR25 6-pos, SW2 FIELD, SW3 SUB, SW4 MINUS, SW5 PLUS

Commit message: Fascia R rev B: J1 is the upright JST B6B-PH-SM4-TB (footprint, 3D model, generator, board, routes)
New TS06_JST_PH_B6B-PH-SM4-TB_Back (KiCad 10's Connector_JST land pattern, mirrored in X for the back, SMD only, no plated
hole) written by tools/mkfp.py; a drawn 3D model for it (the KiCad library has no model for the SM4-TB parts) in
smd_fascia.scad and tools/models3d.json. tools/mkpcb_fascia_rhythm.py puts it where the side-entry part was (between the
buttons, pin order kept, origin y 33.0), D8 and D7 laid into the pads' top ends, A6 / A7 / +5V re-routed from below the tails;
the title block says rev B. KiCad DRC: 0 violations, 0 unconnected, 0 footprint errors. F and the other fascias are untouched.

Co-Authored-By: Claude Opus 5.5 <noreply@anthropic.com>
Claude-Session: https://claude.ai/code/session_01WoV3gyAFgmtuk6W6Dr4bdA
Parts:
- J1: footprint TS06_JST_PH_S6B-PH-SM4-TB_Back -> TS06_JST_PH_B6B-PH-SM4-TB_Back
- moved J1 0.40 mm to (155.4, 33.0)
Routing:
- net +5V: track 215.2 -> 211.4 mm
- net A7: track 98.1 -> 100.5 mm
- net A6: track 102.8 -> 105.3 mm
- net D8: track 32.6 -> 33.4 mm
- net D7: track 5.22 -> 6.02 mm
