File: PCB/TS06-FASCIA-rhythm/TS06-FASCIA-rhythm.kicad_sch (KiCad schematic)
At the start: 14 parts, among them J1 PH 6 SMT, SW1 SR25 6-pos, SW2 LEVER A, SW3 LEVER B, SW4 MINUS, SW5 PLUS

Commit message: Fascia R rev B: J1 is the upright JST B6B-PH-SM4-TB (footprint, 3D model, generator, board, routes)
New TS06_JST_PH_B6B-PH-SM4-TB_Back (KiCad 10's Connector_JST land pattern, mirrored in X for the back, SMD only, no plated
hole) written by tools/mkfp.py; a drawn 3D model for it (the KiCad library has no model for the SM4-TB parts) in
smd_fascia.scad and tools/models3d.json. tools/mkpcb_fascia_rhythm.py puts it where the side-entry part was (between the
buttons, pin order kept, origin y 33.0), D8 and D7 laid into the pads' top ends, A6 / A7 / +5V re-routed from below the tails;
the title block says rev B. KiCad DRC: 0 violations, 0 unconnected, 0 footprint errors. F and the other fascias are untouched.

Co-Authored-By: Claude Opus 5.5 <noreply@anthropic.com>
Claude-Session: https://claude.ai/code/session_01WoV3gyAFgmtuk6W6Dr4bdA
Parts:
- J1: footprint TS06:TS06_JST_PH_S6B-PH-SM4-TB_Back -> TS06:TS06_JST_PH_B6B-PH-SM4-TB_Back
Changed lines of the file:
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@@
 (title "TS06-FASCIA-rhythm - control panel and product face, on the tube grid")
 (date "2026-09-08")
-(rev "A")
+(rev "B")
 (company "TERMINAL-06")
 (comment 1 "Five controls, six wires. Generated by tools/mksch.py")
@@
 )
 )
-(property "Footprint" "TS06:TS06_JST_PH_S6B-PH-SM4-TB_Back"
+(property "Footprint" "TS06:TS06_JST_PH_B6B-PH-SM4-TB_Back"
 (at 238.76 80.01 0)
 (hide yes)
